Commit message: Added kinect with relative rosplugin

File: robots/hand.xacro (robot description, xacro)
@@ -79,4 +79,81 @@
       <mimic joint="${ns}_finger_joint1" />
     </joint>
+    <!-- Adding the kinect link and joint, with relative ros plugin for publishing imgs -->
+    <!-- kinect link -->
+    <link name="${ns}_kinect_link">
+      <!-- <pose>0 0 0.5 0 0 0</pose> -->
+      <inertial>
+        <origin rpy="0 0 0" xyz="0 0 0"/>
+        <mass value="0.00"/>  <!-- Was 0.01 -->
+        <inertia ixx="2.2124416e-03" ixy="-1.2294101e-05" ixz="3.4938785e-05"
+               iyy="2.1193702e-03" iyz="-5.0120904e-06"
+               izz="2.0064271e-03" />
+      </inertial>
+      <collision name="collision">
+        <geometry>
+          <box size="0.073000 0.276000 0.072000"/>
+        </geometry>
+      </collision>
+      <visual name="visual">
+        <geometry>
+          <mesh filename="model://kinect_ros/meshes/kinect.dae"/>  <!-- path should maybe be model://kinect_ros/meshes/kinect.dae -->
+        </geometry>
+      </visual>
+      <!-- sensor -->
+    </link>
+     <!-- <arg name="pi/2" value="1.5707963267948966" /> -->
+    <!-- kinect joint -->
+    <joint name="${ns}_kinect_joint" type="fixed">
+            <origin rpy="0 -1.5707963267948966 3.1415926535" xyz="0.075 0 0.075"/>
+            <parent link="${ns}_hand"/>
+            <child link="${ns}_kinect_link"/>
+            <axis xyz="0 0 0"/>
+    </joint>
+    <!-- Adding kinect ros plugin  -->
+    <gazebo reference="${ns}_kinect_link">
+      <sensor name="camera" type="depth">
+        <update_rate>20</update_rate>
+        <camera>
+          <horizontal_fov>1.047198</horizontal_fov>
+          <image>
+            <width>640</width>
+            <height>480</height>
+            <format>R8G8B8</format>
+          </image>
+          <clip>
+            <near>0.05</near>
+            <far>3</far>
+          </clip>
+        </camera>
+        <!-- plugin -->
+        <!-- Openni camera plugin -->
+        <plugin name="camera_plugin" filename="libgazebo_ros_openni_kinect.so">
+          <baseline>0.2</baseline>
+          <alwaysOn>true</alwaysOn>
+          <!-- Keep this zero, update_rate in the parent <sensor> tag
+            will control the frame rate. -->
+          <updateRate>0.0</updateRate>
+          <cameraName>camera_ir</cameraName>
+          <imageTopicName>/camera/color/image_raw</imageTopicName>
+          <cameraInfoTopicName>/camera/color/camera_info</cameraInfoTopicName>
+          <depthImageTopicName>/camera/depth/image_raw</depthImageTopicName>
+          <depthImageCameraInfoTopicName>/camera/depth/camera_info</depthImageCameraInfoTopicName>
+          <pointCloudTopicName>/camera/depth/points</pointCloudTopicName>
+          <frameName>${ns}_kinect_link</frameName>
+          <pointCloudCutoff>0.5</pointCloudCutoff>
+          <pointCloudCutoffMax>3.0</pointCloudCutoffMax>
+          <distortionK1>0</distortionK1>
+          <distortionK2>0</distortionK2>
+          <distortionK3>0</distortionK3>
+          <distortionT1>0</distortionT1>
+          <distortionT2>0</distortionT2>
+          <CxPrime>0</CxPrime>
+          <Cx>0</Cx>
+          <Cy>0</Cy>
+          <focalLength>0</focalLength>
+          <hackBaseline>0</hackBaseline>
+        </plugin>
+      </sensor>
+    </gazebo>
   </xacro:macro>
 </robot>
